Commit message: Setup plugins to work with real robot (for experiment)

File: muse_ws/src/state_estimator/urdfs/go2_luna_hybrid.urdf (robot description, URDF)
Before this commit: robot go2_luna, 17 links, 16 joints
Links:
- removed link BL_calf
- removed link BL_thigh
- removed link BR_calf
- removed link BR_thigh
- removed link FL_calf
- removed link FL_thigh
- removed link FR_calf
- removed link FR_thigh
- added link BL_lower_leg; collision cylinder length=0.12 radius=0.013; visual cylinder length=0.12 radius=0.013
- added link BL_upper_leg; collision box size=0.213 0.0245 0.034; visual box size=0.213 0.0245 0.034
- added link BR_lower_leg; collision cylinder length=0.12 radius=0.013; visual cylinder length=0.12 radius=0.013
- added link BR_upper_leg; collision box size=0.213 0.0245 0.034; visual box size=0.213 0.0245 0.034
- added link FL_lower_leg; collision cylinder length=0.12 radius=0.012; visual cylinder length=0.12 radius=0.012
- added link FL_upper_leg; collision box size=0.213 0.0245 0.034; visual box size=0.213 0.0245 0.034
- added link FR_lower_leg; collision cylinder length=0.12 radius=0.013; visual cylinder length=0.12 radius=0.013
- added link FR_upper_leg; collision box size=0.213 0.0245 0.034; visual box size=0.213 0.0245 0.034
Joints:
- removed joint BL_calf_joint
- removed joint BL_thigh_joint
- removed joint BR_calf_joint
- removed joint BR_thigh_joint
- removed joint FL_calf_joint
- removed joint FL_thigh_joint
- removed joint FR_calf_joint
- removed joint FR_thigh_joint
- added joint BL_lower_leg_joint: type revolute, parent BL_upper_leg, child BL_lower_leg, origin xyz=0 0 -0.213 rpy=0 0 0, axis 0 1 0, limit lower=-2.7227 upper=-0.83776 effort=12 velocity=10
- added joint BL_upper_leg_joint: type revolute, parent BL_shoulder, child BL_upper_leg, origin xyz=0 0.0955 0 rpy=0 0 0, axis 0 -1 0, limit lower=-1.5708 upper=3.4907 effort=12 velocity=10
- added joint BR_lower_leg_joint: type revolute, parent BR_upper_leg, child BR_lower_leg, origin xyz=0 0 -0.213 rpy=0 0 0, axis 0 -1 0, limit lower=0.83776 upper=2.7227 effort=12 velocity=10
- added joint BR_upper_leg_joint: type revolute, parent BR_shoulder, child BR_upper_leg, origin xyz=0 -0.0955 0 rpy=0 0 0, axis 0 1 0, limit lower=-3.4907 upper=1.5708 effort=12 velocity=10
- added joint FL_lower_leg_joint: type revolute, parent FL_upper_leg, child FL_lower_leg, origin xyz=0 0 -0.213 rpy=0 0 0, axis 0 1 0, limit lower=-2.7227 upper=-0.83776 effort=12 velocity=10
- added joint FL_upper_leg_joint: type revolute, parent FL_shoulder, child FL_upper_leg, origin xyz=0 0.0955 0 rpy=0 0 0, axis 0 -1 0, limit lower=-1.5708 upper=3.4907 effort=12 velocity=10
- added joint FR_lower_leg_joint: type revolute, parent FR_upper_leg, child FR_lower_leg, origin xyz=0 0 -0.213 rpy=0 0 0, axis 0 -1 0, limit lower=0.83776 upper=2.7227 effort=12 velocity=10
- added joint FR_upper_leg_joint: type revolute, parent FR_shoulder, child FR_upper_leg, origin xyz=0 -0.0955 0 rpy=0 0 0, axis 0 1 0, limit lower=-3.4907 upper=1.5708 effort=12 velocity=10
- joint BL_foot_joint: parent BL_calf -> BL_lower_leg
- joint BR_foot_joint: parent BR_calf -> BR_lower_leg
- joint FL_foot_joint: parent FL_calf -> FL_lower_leg
- joint FR_foot_joint: parent FR_calf -> FR_lower_leg

Commit message: Add imu-based odom plugin

File: muse_ws/src/state_estimator/urdfs/go2_luna_hybrid.urdf (robot description, URDF)
Before this commit: robot go2_luna, 17 links, 16 joints
Joints:
- joint BL_lower_leg_joint: origin xyz=0 0 -0.213 rpy=0 0 0 -> xyz=0 0 -0.213 rpy=0 -1.3 0
- joint BR_shoulder_joint: origin xyz=-0.27 -0.0665 0 rpy=0 0 0 -> xyz=-0.27 -0.0665 0 rpy=0 1.3 0
- joint FL_lower_leg_joint: origin xyz=0 0 -0.213 rpy=0 0 0 -> xyz=0 0 -0.213 rpy=0 -1.3 0
- joint FR_lower_leg_joint: origin xyz=0 0 -0.213 rpy=0 0 0 -> xyz=0 0 -0.213 rpy=0 1.3 0

Commit message: Progress experiment

File: muse_ws/src/state_estimator/urdfs/go2_luna_hybrid.urdf (robot description, URDF)
Before this commit: robot go2_luna, 17 links, 16 joints
Links:
- removed link BL_lower_leg
- removed link BL_upper_leg
- removed link BR_lower_leg
- removed link BR_upper_leg
- removed link FL_lower_leg
- removed link FL_upper_leg
- removed link FR_lower_leg
- removed link FR_upper_leg
- added link BL_calf; collision cylinder length=0.12 radius=0.013; visual cylinder length=0.12 radius=0.013
- added link BL_thigh; collision box size=0.213 0.0245 0.034; visual box size=0.213 0.0245 0.034
- added link BR_calf; collision cylinder length=0.12 radius=0.013; visual cylinder length=0.12 radius=0.013
- added link BR_thigh; collision box size=0.213 0.0245 0.034; visual box size=0.213 0.0245 0.034
- added link FL_calf; collision cylinder length=0.12 radius=0.012; visual cylinder length=0.12 radius=0.012
- added link FL_thigh; collision box size=0.213 0.0245 0.034; visual box size=0.213 0.0245 0.034
- added link FR_calf; collision cylinder length=0.12 radius=0.013; visual cylinder length=0.12 radius=0.013
- added link FR_thigh; collision box size=0.213 0.0245 0.034; visual box size=0.213 0.0245 0.034
Joints:
- removed joint BL_lower_leg_joint
- removed joint BL_upper_leg_joint
- removed joint BR_lower_leg_joint
- removed joint BR_upper_leg_joint
- removed joint FL_lower_leg_joint
- removed joint FL_upper_leg_joint
- removed joint FR_lower_leg_joint
- removed joint FR_upper_leg_joint
- added joint BL_calf_joint: type revolute, parent BL_thigh, child BL_calf, origin xyz=0 0 -0.213 rpy=0 0 0, axis 0 1 0, limit lower=-2.7227 upper=-0.83776 effort=12 velocity=10
- added joint BL_thigh_joint: type revolute, parent BL_shoulder, child BL_thigh, origin xyz=0 0.0955 0 rpy=0 0 0, axis 0 -1 0, limit lower=-1.5708 upper=3.4907 effort=12 velocity=10
- added joint BR_calf_joint: type revolute, parent BR_thigh, child BR_calf, origin xyz=0 0 -0.213 rpy=0 0 0, axis 0 -1 0, limit lower=0.83776 upper=2.7227 effort=12 velocity=10
- added joint BR_thigh_joint: type revolute, parent BR_shoulder, child BR_thigh, origin xyz=0 -0.0955 0 rpy=0 0 0, axis 0 1 0, limit lower=-3.4907 upper=1.5708 effort=12 velocity=10
- added joint FL_calf_joint: type revolute, parent FL_thigh, child FL_calf, origin xyz=0 0 -0.213 rpy=0 0 0, axis 0 1 0, limit lower=-2.7227 upper=-0.83776 effort=12 velocity=10
- added joint FL_thigh_joint: type revolute, parent FL_shoulder, child FL_thigh, origin xyz=0 0.0955 0 rpy=0 0 0, axis 0 -1 0, limit lower=-1.5708 upper=3.4907 effort=12 velocity=10
- added joint FR_calf_joint: type revolute, parent FR_thigh, child FR_calf, origin xyz=0 0 -0.213 rpy=0 0 0, axis 0 -1 0, limit lower=0.83776 upper=2.7227 effort=12 velocity=10
- added joint FR_thigh_joint: type revolute, parent FR_shoulder, child FR_thigh, origin xyz=0 -0.0955 0 rpy=0 0 0, axis 0 1 0, limit lower=-3.4907 upper=1.5708 effort=12 velocity=10
- joint BL_foot_joint: parent BL_lower_leg -> BL_calf
- joint BR_foot_joint: parent BR_lower_leg -> BR_calf
- joint BR_shoulder_joint: origin xyz=-0.27 -0.0665 0 rpy=0 1.3 0 -> xyz=-0.27 -0.0665 0 rpy=0 0 0
- joint FL_foot_joint: parent FL_lower_leg -> FL_calf
- joint FR_foot_joint: parent FR_lower_leg -> FR_calf
